Commit message: updated gripper

File: robot_model/right_eef.urdf.xacro (robot description, xacro)
@@ -62,5 +62,5 @@
     </link>
     <joint name="right_tcp_joint" type="fixed">
-      <origin xyz="0 0 0.15" rpy="0 0 0" />
+      <origin xyz="0 0 0.14" rpy="0 0 0" />
       <parent link="gripper_link"/>
       <child link="right_tcp"/>

Commit message: updated tcp

File: robot_model/right_eef.urdf.xacro (robot description, xacro)
@@ -61,4 +61,5 @@
         </collision>
     </link>
+    <!-- <xacro:if value="${sim}"> -->
     <joint name="right_tcp_joint" type="fixed">
       <origin xyz="0 0 0.14" rpy="0 0 0" />
@@ -67,4 +68,14 @@
     </joint>
     <link name="right_tcp" />
+    <!-- </xacro:if> -->
+    <!-- 20251117 hand-eye calibration result -->
+    <!-- <xacro:unless value="${sim}">
+      <joint name="right_tcp_joint" type="fixed">
+        <origin xyz="0.08855604 -0.03328494 -0.11521747" rpy="-0.0104157 -0.0006242 1.5653368" />
+        <parent link="right_camera_color_optical_frame"/>
+        <child link="right_tcp"/>
+      </joint>
+      <link name="right_tcp" />
+    </xacro:unless> -->
   </xacro:macro>
 </robot>

File: urdf/dual_arm_robot.urdf.xacro (robot description, xacro)
@@ -50,7 +50,4 @@
       can_interface_right="${right_arm_can_interface}"
       namespace="upper_orin" />
-    <xacro:left_eef name="${left_eef_name}" parent="link7_left">
-      <origin xyz="0 0.0335 0" rpy="0 0 0"/>
-    </xacro:left_eef>
     <xacro:sensor_d435
       parent="${left_eef_name}_camera_base_link"
@@ -59,7 +56,7 @@
       <origin xyz="0 0 0" rpy="0 0 0"/>
     </xacro:sensor_d435>
-    <xacro:right_eef name="${right_eef_name}" parent="link7_right">
-      <origin xyz="0 0.0335 0" rpy="0 ${M_PI} 0"/>
-    </xacro:right_eef>
+    <xacro:left_eef name="${left_eef_name}" parent="link7_left">
+      <origin xyz="0 0.0335 0" rpy="0 0 0"/>
+    </xacro:left_eef>
     <xacro:sensor_d435
       parent="${right_eef_name}_camera_base_link"
@@ -68,4 +65,7 @@
       <origin xyz="0 0 0" rpy="0 0 0"/>
     </xacro:sensor_d435>
+    <xacro:right_eef name="${right_eef_name}" parent="link7_right">
+      <origin xyz="0 0.0335 0" rpy="0 ${M_PI} 0"/>
+    </xacro:right_eef>
   </xacro:macro>
 </robot>
