Commit message: updated models

File: robot_model/left_eef.urdf.xacro (robot description, xacro)
@@ -48,5 +48,5 @@
         <origin xyz="0 0 0" rpy="${M_PI_2} 0 ${M_PI}" />
         <geometry>
-          <mesh filename="package://dual_arm_robot/meshes/visual/KD-ES70A-Z1-24V.STL" scale="0.001 0.001 0.001"/>
+          <mesh filename="package://dual_arm_robot/meshes/visual/KD-ES70A-Z1-24V.STL" />
         </geometry>
         <material name="">
@@ -57,14 +57,15 @@
         <origin xyz="0 0 0" rpy="${M_PI_2} 0 ${M_PI}" />
         <geometry>
-          <mesh filename="package://dual_arm_robot/meshes/collision/KD-ES70A-Z1-24V.STL" scale="0.001 0.001 0.001"/>
+          <mesh filename="package://dual_arm_robot/meshes/collision/KD-ES70A-Z1-24V.STL" />
         </geometry>
         </collision>
     </link>
     <joint name="left_tcp_joint" type="fixed">
-      <origin xyz="0 0.12 0" rpy="-${M_PI_2} 0 0" />
+      <origin xyz="0 0.135 0" rpy="-${M_PI_2} 0 0" />
       <parent link="suction_cup_link"/>
       <child link="left_tcp"/>
     </joint>
-    <link name="left_tcp" >
+    <link name="left_tcp" />
+    <!-- <link name="left_tcp" >
       <visual>
         <origin rpy="0 0 0" xyz="0 0 -0.0375" />
@@ -82,5 +83,5 @@
         </geometry>
       </collision>
-    </link>
+    </link> -->
   </xacro:macro>
 </robot>
